File: hardware/adcs_board/adcs_board.kicad_pcb (KiCad board)
At the start: 4 copper layers, 89.1 x 92.2 mm, 157 parts, among them IC1 STM32F411VCT6, J1 472192001, J5 2053380006, J6 5055671081, J7 2053380006, J8 MTLW-104-05-G-S-170-ND, T3 IRF7105TR, T4 IRF7105TR, U1 MCP2515-E/ML, U18 AMS1117-3.3, U19 A3G4250D, U2 TMCS1101A3BQDRQ1, U20 TMCS1101A3BQDRQ1, U22 SN65HVD230DR, U23 ADS1257IRGWT, U24 REF5025AID, U25 HMC1002-TR, U26 LM324NSR, U27 HMC1001-RC, U28 ADS1257IRGWT, U29 LM324NSR, U3 TMCS1101A3BQDRQ1, U30 DRV8833RTYR, U31 DRV8833RTYR, U4 TMCS1101A3BQDRQ1, U5 MT3608, U6 MT3608, Y1 ABLS-8.000MHZ-B2-T

Commit message: hardware: schematic and layout fixes
Parts:
- added R54: 4,7k, Resistor_SMD:R_0402_1005Metric_Pad0.72x0.64mm_HandSolder, F.Cu at (159.5, 110.5)
- added R7: 4,7k, Resistor_SMD:R_0402_1005Metric_Pad0.72x0.64mm_HandSolder, F.Cu at (159.5, 109.0)
- C68: value GRM155R60J106ME15D -> C0402C103K5RECAUTO
- C69: value GRM155R60J106ME15D -> CL05B104KP5NNNC
- moved R4 31.9 mm to (172.9, 125.6)
- moved C7 31.9 mm to (172.9, 120.3)
- moved R3 31.9 mm to (172.9, 122.9)
- moved L1 31.2 mm to (168.0, 126.0)
- moved C8 14.8 mm to (172.9, 131.0)
- moved C52 14.8 mm to (170.2, 84.8)
- moved C62 14.8 mm to (183.4, 65.6)
- moved C64 14.8 mm to (183.4, 63.0)
- moved C73 14.8 mm to (173.2, 95.5)
- moved C74 14.8 mm to (173.2, 89.3)
- moved C82 14.8 mm to (185.6, 94.2)
- moved C91 14.8 mm to (143.2, 120.3)
- moved C92 14.8 mm to (143.2, 118.0)
- moved D6 14.8 mm to (175.4, 71.3)
- moved FB2 14.8 mm to (179.5, 64.3)
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Connections:
- net /NRST renamed /mcu/NRST
- net /mcu_circuits/SS_AIN0 renamed /SS_AIN0
- net /mcu_circuits/SS_AIN1 renamed /SS_AIN1
- net /mcu_circuits/coarse_sun-sensor1/REFP renamed /coarse_sun-sensor1/REFP
- net /mcu_circuits/magnetometer1/S/R1 renamed /magnetometer1/S/R1
- net /mcu_circuits/magnetometer1/S/R2 renamed /magnetometer1/S/R2
- net /mcu_circuits/magnetometer1/out+1001 renamed /magnetometer1/out+1001
- net /mcu_circuits/magnetometer1/out+b renamed /magnetometer1/out+b
- net /mcu_circuits/magnetometer1/out-b renamed /magnetometer1/out-b
- net /mcu_circuits/magnetometer1/outx renamed /magnetometer1/outx
- net /mcu_circuits/magnetometer1/outy renamed /magnetometer1/outy
- net /mcu_circuits/magnetometer1/outz renamed /magnetometer1/outz
- net /mcu_circuits/magnetometer1/vdd_div renamed /magnetometer1/vdd_div
- net /mcu_circuits/magnetometer1/vref renamed /magnetometer1/vref
- net /mcu_circuits/magnetorquer control1/bout1u7 renamed /magnetorquer control1/bout1u7
- net /mcu_circuits/magnetorquer control1/bout2u7 renamed /magnetorquer control1/bout2u7
- net /mcu_circuits/magnetorquer control1/current_sensingx renamed /magnetorquer control1/current_sensingx
- net /mcu_circuits/magnetorquer control1/current_sensingy renamed /magnetorquer control1/current_sensingy
- net /mcu_circuits/magnetorquer control1/current_sensingz renamed /magnetorquer control1/current_sensingz
- net /mcu_circuits/magnetorquerx renamed /magnetorquerx
- net /mcu_circuits/magnetorquerx2 renamed /magnetorquerx2
- net /mcu_circuits/magnetorquery renamed /magnetorquery
- net /mcu_circuits/magnetorquery2 renamed /magnetorquery2
- net /mcu_circuits/magnetorquerz renamed /magnetorquerz
- net /mcu_circuits/magnetorquerz2 renamed /magnetorquerz2
- C7 pad 1: /mcu_circuits/magnetometer1/8v -> /magnetometer1/8v(2)
- C9 pad 1: /mcu_circuits/magnetometer1/8v(2) -> /magnetometer1/8v
- D1 pad 1: /mcu_circuits/magnetometer1/8v(2) -> /magnetometer1/8v(2)
- D2 pad 1: /mcu_circuits/magnetometer1/8v -> /magnetometer1/8v
- L1 pad 2: Net-(D2-A) -> Net-(D1-A)
- L2 pad 2: Net-(D1-A) -> Net-(D2-A)
- R3 pad 1: /mcu_circuits/magnetometer1/8v -> /magnetometer1/8v(2)
- R3 pad 2: Net-(U5-FB) -> Net-(U6-FB)
- R4 pad 1: Net-(U5-FB) -> Net-(U6-FB)
- R5 pad 1: /mcu_circuits/magnetometer1/8v(2) -> /magnetometer1/8v
- R5 pad 2: Net-(U6-FB) -> Net-(U5-FB)
- R6 pad 1: Net-(U6-FB) -> Net-(U5-FB)
- R90 pad 2: /mcu_circuits/magnetometer1/8v -> /magnetometer1/8v
- R92 pad 2: /mcu_circuits/magnetometer1/8v(2) -> /magnetometer1/8v(2)
Routing:
- net /magnetometer1/8v(2): track 0.00 -> 22.7 mm, vias 0 -> 1
- net /mcu_circuits/magnetometer1/8v(2): track 22.4 -> 0.00 mm, vias 1 -> 0
- net /mcu_circuits/magnetometer1/8v: track 11.9 -> 0.00 mm, vias 1 -> 0
- net /magnetometer1/8v: track 0.00 -> 11.6 mm, vias 0 -> 1
- net +3V3: track 89.3 -> 100.4 mm, vias 30 -> 34
- net /GYRO_I2C_SDL: track 10.7 -> 14.4 mm
- net Net-(U6-FB): track 12.4 -> 14.4 mm
- net Net-(U5-FB): track 11.9 -> 13.9 mm
- net /GYRO_I2C_SDA: track 14.7 -> 16.4 mm
- net /SD_SPI_MOSI: track 48.4 -> 46.7 mm
- net /SD_SPI_SS: track 46.4 -> 46.9 mm
