File: hardware/adcs_board/adcs_board.kicad_sch (KiCad schematic)
At the start: 3 parts, among them IC1 STM32F411VCT6

Commit message: hardware: schematic and layout fixes
Parts:
- removed C1: 100nF, Capacitor_SMD:C_0402_1005Metric_Pad0.74x0.62mm_HandSolder, symbol Device:C
- removed IC1: STM32F411VCT6, adcs_board:QFP50P1600X1600X160-100N, symbol adcs_board:STM32F411VCT6
- removed R1: 10k, Resistor_SMD:R_0402_1005Metric_Pad0.72x0.64mm_HandSolder, symbol Device:R
Connections:
- no-connect marks 41 -> 2
Other:
- added sheet coarse_sun-sensor1 (corsesunsensor.kicad_sch)
- added sheet magnetometer1 (magnetometer.kicad_sch)
- added sheet magnetorquer control1 (hcp_sch.kicad_sch)
- added sheet mcu (mcu.kicad_sch)
- sheet mcu_circuits ports: added SS_AIN0, SS_AIN1, magnetorquerx, magnetorquerx2, magnetorquery, magnetorquery2, magnetorquerz, magnetorquerz2; removed AIN1u7, AIN1u8, AIN2u7, AIN2u8, BIN1u7, BIN1u8, BIN2u7, BIN2u8, MAG_CS_SS, MAG_INT, MAG_I/O_CLOCK, MAG_SPI_MISO, MAG_SPI_MOSI, MAG_SPI_SCK, SRI_IN, SRI_IN2, SS_CS, SS_INT, SS_I/O_CLOCK, SS_SPI_MISO, SS_SPI_MOSI, SS_SPI_SCK, currentcoilx, currentcoily, currentcoilz, nfaultu7, nfaultu8, nsleepu7, nsleepu8
