File: hardware/adcs_board/corsesunsensor.kicad_sch (KiCad schematic)
At the start: 24 parts, among them U23 ADS1257IRGWT, U24 REF5025AID

Commit message: Update and fix part number issues
Parts:
- C83: footprint Capacitor_SMD:C_0402_1005Metric_Pad0.74x0.62mm_HandSolder -> Capacitor_SMD:C_0603_1608Metric
- U23: MF (none) -> Texas Instruments
- U24: Availability In Stock -> (none); Check_prices https://www.snapeda.com/parts/REF5025AID/Texas+Instruments/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 -> (none); Description_1 2.5-V, 3-µVpp/V noise, 3-ppm/°C drift precision series volt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 -> (none); MP REF5025AID -> (none); Package SOIC-8 Texas Instruments -> (none); Price None -> (none); Purchase-URL https://www.snapeda.com/api/url_track_click_mouser/?unipart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 -> (none); SnapEDA_Link https://www.snapeda.com/parts/REF5025AID/Texas+Instruments/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 -> (none)
Changed lines of the file:
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@@
 	(label "REFP"
 		(at 85.09 126.365 0)
-		(fields_autoplaced yes)
 		(effects
 			(font
@@
 	(label "REFP"
 		(at 81.28 54.61 0)
-		(fields_autoplaced yes)
 		(effects
 			(font
@@
 		(shape input)
 		(at 148.59 49.53 0)
-		(fields_autoplaced yes)
 		(effects
 			(font
@@
 		(shape input)
 		(at 49.53 85.09 180)
-		(fields_autoplaced yes)
 		(effects
 			(font
@@
 		(shape input)
 		(at 49.53 77.47 180)
-		(fields_autoplaced yes)
 		(effects
 			(font
@@
 		(shape input)
 		(at 49.53 64.77 180)
-		(fields_autoplaced yes)
 		(effects
 			(font
@@
 		(shape input)
 		(at 148.59 74.93 0)
-		(fields_autoplaced yes)
 		(effects
 			(font
@@
 		(shape input)
 		(at 147.32 44.45 0)
-		(fields_autoplaced yes)
 		(effects
 			(font
@@
 		(shape input)
 		(at 148.59 68.58 0)
-		(fields_autoplaced yes)
 		(effects
 			(font
@@
 		(shape input)
 		(at 49.53 73.66 180)
-		(fields_autoplaced yes)
 		(effects
 			(font
@@
 		(shape input)
 		(at 148.59 55.88 0)
-		(fields_autoplaced yes)
 		(effects
 			(font
@@
 		(shape input)
 		(at 148.59 62.23 0)
-		(fields_autoplaced yes)
 		(effects
 			(font
@@
 			)
 		)
-		(property "Datasheet" ""
+		(property "Datasheet" "https://www.ti.com/general/docs/suppproductinfo.tsp?distId=10&gotoUrl=https%3A%2F%2Fwww.ti.com%2Flit%2Fgpn%2Fref5020"
 			(at 116.205 118.745 0)
 			(effects
@@
 			)
 		)
-		(property "Description" ""
+		(property "Description" "IC VREF SERIES 0.1% 8SOIC"
 			(at 116.205 118.745 0)
 			(effects
@@
 		)
 		(property "MF" "Texas Instruments"
-			(at 116.205 118.745 0)
-			(effects
-				(font
-					(size 1.27 1.27)
-				)
-				(justify bottom)
-				(hide yes)
-			)
-		)
-		(property "Description_1" "\n2.5-V, 3-µVpp/V noise, 3-ppm/°C drift precision series voltage reference\n"
-			(at 116.205 118.745 0)
-			(effects
-				(font
-					(size 1.27 1.27)
-				)
-				(justify bottom)
-				(hide yes)
-			)
-		)
-		(property "Package" "SOIC-8 Texas Instruments"
-			(at 116.205 118.745 0)
-			(effects
-				(font
-					(size 1.27 1.27)
-				)
-				(justify bottom)
-				(hide yes)
-			)
-		)
-		(property "Price" "None"
-			(at 116.205 118.745 0)
-			(effects
-				(font
-					(size 1.27 1.27)
-				)
-				(justify bottom)
-				(hide yes)
-			)
-		)
-		(property "SnapEDA_Link" "https://www.snapeda.com/parts/REF5025AID/Texas+Instruments/view-part/?ref=snap"
-			(at 116.205 118.745 0)
-			(effects
-				(font
-					(size 1.27 1.27)
-				)
-				(justify bottom)
-				(hide yes)
-			)
-		)
-		(property "MP" "REF5025AID"
-			(at 116.205 118.745 0)
-			(effects
-				(font
-					(size 1.27 1.27)
-				)
-				(justify bottom)
-				(hide yes)
-			)
-		)
-		(property "Purchase-URL" "https://www.snapeda.com/api/url_track_click_mouser/?unipart_id=98520&manufacturer=Texas Instruments&part_name=REF5025AID&search_term=None"
-			(at 116.205 118.745 0)
-			(effects
-				(font
-					(size 1.27 1.27)
-				)
-				(justify bottom)
-				(hide yes)
-			)
-		)
-		(property "Availability" "In Stock"
-			(at 116.205 118.745 0)
-			(effects
-				(font
-					(size 1.27 1.27)
-				)
-				(justify bottom)
-				(hide yes)
-			)
-		)
-		(property "Check_prices" "https://www.snapeda.com/parts/REF5025AID/Texas+Instruments/view-part/?ref=eda"
 			(at 116.205 118.745 0)
 			(effects
@@
 			)
 		)
-		(property "Footprint" "Capacitor_SMD:C_0402_1005Metric_Pad0.74x0.62mm_HandSolder"
+		(property "Footprint" "Capacitor_SMD:C_0603_1608Metric"
 			(at 94.9452 135.89 0)
 			(effects
@@
 			)
 		)
-		(property "Datasheet" "ADS1257IRGWT"
+		(property "Datasheet" "https://www.ti.com/general/docs/suppproductinfo.tsp?distId=10&gotoUrl=https%3A%2F%2Fwww.ti.com%2Flit%2Fgpn%2Fads1257"
 			(at 111.76 62.23 0)
 			(effects
@@
 			)
 		)
-		(property "Description" ""
+		(property "Description" "IC ADC 24BIT SIGMA-DELTA 20VQFN"
 			(at 111.76 62.23 0)
 			(effects
+				(font
+					(size 1.27 1.27)
+				)
+				(hide yes)
+			)
+		)
+		(property "MF" "Texas Instruments"
+			(at 111.76 62.23 0)
+			(effects

Commit message: hardware: schematic and layout fixes
Other:
- moved on the sheet: C72, C73, C74, C75, C76, C77, C78, C79, C80, C81, C82, C83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
