File: hardware/adcs_board/mcu_circuits.kicad_sch (KiCad schematic)
At the start: 44 parts, among them J1 472192001, J5 2053380006, J6 5055671081, J7 2053380006, J8 MTLW-104-05-G-S-170-ND, U1 MCP2515-E/ML, U18 AMS1117-3.3, U19 A3G4250D, U20 TMCS1101A3BQDRQ1, U22 SN65HVD230DR, Y1 ABLS-8.000MHZ-B2-T

Commit message: Update and fix part number issues
Parts:
- C52, C54: footprint Capacitor_SMD:C_0402_1005Metric_Pad0.74x0.62mm_HandSolder -> Capacitor_SMD:C_0603_1608Metric
- C68: value GRM155R60J106ME15D -> C0402C103K5RECAUTO; Availability In Stock -> (none); Check_prices https://www.snapeda.com/parts/GRM155R60J106ME15D/Murata+Ele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 -> (none); MF Murata -> KEMET; MP GRM155R60J106ME15D -> (none); Package 1005 Murata -> (none); Price None -> (none); Purchase-URL https://www.snapeda.com/api/url_track_click_mouser/?unipart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 -> (none); SnapEDA_Link https://www.snapeda.com/parts/GRM155R60J106ME15D/Murata+Ele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 -> (none)
- C69: value GRM155R60J106ME15D -> CL05B104KP5NNNC; Availability In Stock -> (none); Check_prices https://www.snapeda.com/parts/885012206071/Wurth+Electronic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 -> (none); MF Wurth Electronics Inc -> Samsung Electro-Mechanics; MP 885012206071 -> (none); Package 0603 Wurth Electronics -> (none); Price None -> (none); Purchase-URL https://www.snapeda.com/api/url_track_click_mouser/?unipart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 -> (none); SnapEDA_Link https://www.snapeda.com/parts/885012206071/Wurth+Electronic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 -> (none)
- J1: MF (none) -> Molex
- U1: MF (none) -> Microchip Technology
- U18: MF (none) -> EVVO
- U19: MF (none) -> STMicroelectronics
- U20: MF (none) -> Texas Instruments
- XTAL1: MF (none) -> Abracon LLC
- Y1: Availability In Stock -> (none); Check_prices https://www.snapeda.com/parts/ABLS-8.000MHZ-B2-T/Abracon/vi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 -> (none); Description_1 CRYSTAL 8.0000MHZ 18PF SMD / AB Series HC49U Crystals, ABLS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 -> (none); MANUFACTURER Abracon -> (none); MAXIMUM_PACKAGE_HEIGHT 4.2 mm -> (none); MP ABLS-8.000MHZ-B2-T -> (none); PARTREV 02.16.2021 -> (none); Package None -> (none); Price None -> (none); STANDARD Manufacturer Recommendations -> (none); SnapEDA_Link https://www.snapeda.com/parts/ABLS-8.000MHZ-B2-T/Abracon/vi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 -> (none)

Commit message: hardware: schematic and layout fixes
Parts:
- added R54, R7: 4,7k, Resistor_SMD:R_0402_1005Metric_Pad0.72x0.64mm_HandSolder, symbol Device:R
Connections:
- net +3V3: now also R54.2, R7.2
- net GYRO_I2C_SDA: now also R7.1
- net GYRO_I2C_SDL: now also R54.1
- no-connect marks 17 -> 15
Other:
- removed sheet coarse_sun-sensor1
- removed sheet magnetometer1
- removed sheet magnetorquer control1
