File: hardware/ADCS_bdot/MCU_STM32F7.kicad_sch (KiCad schematic)
At the start: 33 parts, among them IC1 STM32F746ZGT6, IC3 DRV8833RTYR, IC4 DRV8833RTYR, IC5 HMC1001-RC, SW1 SW_Push, U2 TMCS1101A3BQDRQ1, U4 TMCS1101A3BQDRQ1, U5 TMCS1101A3BQDRQ1, U6 HMC1002-TR, Y1 ABM3-8.000MHZ-B4Y-T, Y2 CM7V-T1A-32.768kHz-7pF-10PPM-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

Commit message: add:STM32F4
Parts:
- removed unit 3 of IC1
- removed unit 2 of IC1
- added U7: STM32F413ZHJ6, Footprintlib_adcs_bdot:UFBGA144-10x10mm, symbol Symbollib_adcs_bdot:STM32F413ZHJ6
